Commit message: modify tcp

File: src/franka_softhand/franka_softhand_description/urdf/franka_softhand.urdf.xacro (robot description, xacro)
@@ -42,5 +42,5 @@
   <!-- End-effector frame (TCP) della softhand, riferito a panda_link8 -->
   <joint name="$(arg hand_namespace)_ee_joint" type="fixed">
-    <origin xyz="0.21 -0.05 0.065" rpy="0 0 0"/>
+    <origin xyz="0.18 -0.035 0.065" rpy="0 0 0"/>
     <parent link="$(arg arm_id)_link8"/>
     <child  link="$(arg hand_namespace)_tcp"/>
